Commit message: complete_task06

File: ex03/robot_description/urdf/gazebo.urdf.xacro (robot description, xacro)
@@ -31,4 +31,7 @@
             <odom_publish_frequency>10</odom_publish_frequency>
         </plugin>
+        <plugin filename="gz-sim-imu-system"
+        name="gz::sim::systems::Imu">
+        </plugin>
     </gazebo>
 </robot>

File: ex04/robot_description/urdf/gazebo.urdf.xacro (robot description, xacro)
@@ -2,4 +2,19 @@
 <robot xmlns:xacro="http://www.ros.org/wiki/xacro">
     <gazebo>
+        <!--plugin
+            filename="gz-sim-pose-publisher-system"
+            name="gz::sim::systems::PosePublisher">
+            <publish_link_pose>true</publish_link_pose>
+            <use_pose_vector_msg>true</use_pose_vector_msg>
+            <static_publisher>true</static_publisher>
+            <static_update_frequency>1</static_update_frequency>
+        </plugin-->
+        <!--plugin
+            filename="gz-sim-odometry-publisher-system"
+            name="gz::sim::systems::OdometryPublisher">
+            <odom_frame>robot/odom</odom_frame>
+            <robot_base_frame>robot/base_link</robot_base_frame>
+            <odom_publish_frequency>50</odom_publish_frequency>
+        </plugin-->
         <plugin
             filename="gz-sim-joint-state-publisher-system"
@@ -16,4 +31,7 @@
             <odom_publish_frequency>10</odom_publish_frequency>
         </plugin>
+        <plugin filename="gz-sim-imu-system"
+        name="gz::sim::systems::Imu">
+        </plugin>
     </gazebo>
 </robot>

File: ex04/robot_description/urdf/robot.urdf.xacro (robot description, xacro)
@@ -1,45 +1,80 @@
 <?xml version="1.0" ?>
-<robot name='two_wheeled_stick_robot' xmlns:xacro="http://ros.org/wiki/xacro">
-    <xacro:property name="stick_length" value="0.5"/>
-    <xacro:property name="stick_radius" value="0.02"/>
-    <xacro:property name="wheel_radius" value="0.1"/>
+<robot name='robot' xmlns:xacro="http://ros.org/wiki/xacro">
+    <xacro:include filename="gazebo.urdf.xacro" />
+    <xacro:include filename="lidar.urdf.xacro"/>
+    <xacro:include filename="depth.urdf.xacro" />
+    <xacro:include filename="imu.urdf.xacro" />
+    <xacro:property name="chassis_length" value="0.335"/>
+    <xacro:property name="chassis_width" value="0.265"/>
+    <xacro:property name="chassis_height" value="0.138"/>
+    <xacro:property name="wheel_radius" value="0.033"/>
     <xacro:property name="wheel_thickness" value="0.026"/>
     <xacro:property name="wheel_mass" value="0.05"/>
-    <xacro:property name="wheel_offset_y" value="${stick_length / 2}"/>
+    <xacro:property name="wheel_offset_x" value="0.226"/>
+    <xacro:property name="wheel_offset_y" value="0.1485"/>
+    <xacro:property name="wheel_offset_z" value="0.01"/>
+    <xacro:property name="caster_wheel_radius" value="0.01"/>
+    <xacro:property name="caster_wheel_mass" value="0.01"/>
+    <xacro:property name="caster_wheel_offset_x" value="0.075"/>
+    <xacro:property name="caster_wheel_offset_z" value="${wheel_offset_z - wheel_radius + caster_wheel_radius}"/>
     <xacro:property name="mass" value="1.0"/>
+    <material name="white">
+        <color rgba="1 1 1 1" />
+    </material>
+    <material name="orange">
+        <color rgba="1 0.3 0.1 1"/>
+    </material>
     <material name="blue">
         <color rgba="0.2 0.2 1 1"/>
     </material>
-    <material name="white">
-        <color rgba="1 1 1 1"/>
+    <material name="black">
+        <color rgba="0 0 0 1"/>
     </material>
-    <!-- Stick structure -->
-    <link name="stick">
-        <inertial>
-            <origin xyz="0 0 0" rpy="0 0 0"/>
-            <mass value="${mass}" />
-            <inertia ixx="0.001" ixy="0.0" ixz="0.0"
-                     iyy="0.001" iyz="0.0"
-                     izz="0.001"/>
-        </inertial>
-        <visual>
-            <origin xyz="0 0 0"/>
-            <geometry>
-                <cylinder radius="${stick_radius}" length="${stick_length}"/>
-            </geometry>
-            <material name="white"/>
-        </visual>
-        <collision>
-            <origin xyz="0 0 0"/>
-            <geometry>
-                <cylinder radius="${stick_radius}" length="${stick_length}"/>
-            </geometry>
-        </collision>
+    <material name="red">
+        <color rgba="1 0 0 1"/>
+    </material>
+    <link name="base_link">
     </link>
-    <!-- Left Wheel -->
+    <link name="base_footprint">
+    </link>
+    <joint name="base_footprint_joint" type="fixed">
+        <parent link="base_link"/>
+        <child link="base_footprint"/>
+        <origin xyz="0 0 -0.138" rpy="0 0 0"/>
+    </joint>
+    <joint name="chassis_joint" type="fixed">
+        <parent link="base_link"/>
+        <child link="chassis"/>
+        <origin xyz="${-wheel_offset_x} 0 ${-wheel_offset_z}"/>
+    </joint>
+    <link name='chassis'>
+    <inertial>
+        <origin xyz="${chassis_length/2} 0 ${chassis_height/2}" rpy="0 0 0"/>
+        <mass value="${mass}" />
+        <inertia ixx="${(1/12) * mass * (chassis_width*chassis_width+chassis_height*chassis_height)}" ixy="0.0" ixz="0.0"
+                 iyy="${(1/12) * mass * (chassis_length*chassis_length+chassis_height*chassis_height)}" iyz="0.0"
+                 izz="${(1/12) * mass * (chassis_length*chassis_length+chassis_width*chassis_width)}" />
+    </inertial>
+    <visual>
+        <origin xyz="${chassis_length/2} 0 ${chassis_height/2}"/>
+        <geometry>
+            <box size="${chassis_length} ${chassis_width} ${chassis_height}"/>
+        </geometry>
+        <material name="orange"/>
+    </visual>
+    <collision>
+        <origin xyz="${chassis_length/2} 0 ${chassis_height/2}"/>
+        <geometry>
+            <box size="${chassis_length} ${chassis_width} ${chassis_height}"/>
+        </geometry>
+    </collision>
+    </link>
+    <gazebo reference="chassis">
+        <material>Gazebo/Orange</material>
+    </gazebo>
     <joint name="left_wheel_joint" type="continuous">
-        <parent link="stick"/>
+        <parent link="base_link"/>
         <child link="left_wheel"/>
-        <origin xyz="0 ${wheel_offset_y} 0" rpy="0 0 0"/>
+        <origin xyz="0 ${wheel_offset_y} 0" rpy="-${pi/2} 0 0" />
         <axis xyz="0 0 1"/>
     </joint>
@@ -53,5 +88,5 @@
         <collision>
             <geometry>
-                <cylinder radius="${wheel_radius}" length="${wheel_thickness}"/>
+                <sphere radius="${wheel_radius}"/>
             </geometry>
         </collision>
@@ -59,14 +94,16 @@
             <origin xyz="0 0 0" rpy="0 0 0"/>
             <mass value="${wheel_mass}" />
-            <inertia ixx="0.001" ixy="0.0" ixz="0.0"
-                     iyy="0.001" iyz="0.0"
-                     izz="0.001"/>
+            <inertia ixx="${(1/12) * wheel_mass * (3*wheel_radius*wheel_radius + wheel_thickness*wheel_thickness)}" ixy="0.0" ixz="0.0"
+                     iyy="${(1/12) * wheel_mass * (3*wheel_radius*wheel_radius + wheel_thickness*wheel_thickness)}" iyz="0.0"
+                     izz="${(1/2) * wheel_mass * (wheel_radius*wheel_radius)}" />
         </inertial>
     </link>
-    <!-- Right Wheel -->
+    <gazebo reference="left_wheel">
+        <material>Gazebo/Blue</material>
+    </gazebo>
     <joint name="right_wheel_joint" type="continuous">
-        <parent link="stick"/>
+        <parent link="base_link"/>
         <child link="right_wheel"/>
-        <origin xyz="0 ${-wheel_offset_y} 0" rpy="0 0 0"/>
+        <origin xyz="0 ${-wheel_offset_y} 0" rpy="${pi/2} 0 0" />
         <axis xyz="0 0 -1"/>
     </joint>
@@ -80,5 +117,5 @@
         <collision>
             <geometry>
-                <cylinder radius="${wheel_radius}" length="${wheel_thickness}"/>
+                <sphere radius="${wheel_radius}"/>
             </geometry>
         </collision>
@@ -86,8 +123,41 @@
             <origin xyz="0 0 0" rpy="0 0 0"/>
             <mass value="${wheel_mass}" />
-            <inertia ixx="0.001" ixy="0.0" ixz="0.0"
-                     iyy="0.001" iyz="0.0"
-                     izz="0.001"/>
+            <inertia ixx="${(1/12) * wheel_mass * (3*wheel_radius*wheel_radius + wheel_thickness*wheel_thickness)}" ixy="0.0" ixz="0.0"
+                     iyy="${(1/12) * wheel_mass * (3*wheel_radius*wheel_radius + wheel_thickness*wheel_thickness)}" iyz="0.0"
+                     izz="${(1/2) * wheel_mass * (wheel_radius*wheel_radius)}" />
         </inertial>
     </link>
+    <gazebo reference="right_wheel">
+        <material>Gazebo/Blue</material>
+    </gazebo>
+    <joint name="caster_wheel_joint" type="fixed">
+        <parent link="chassis"/>
+        <child link="caster_wheel"/>
+        <origin xyz="${caster_wheel_offset_x} 0 ${caster_wheel_offset_z}"/>
+    </joint>
+    <link name="caster_wheel">
+        <visual>
+            <geometry>
+                <sphere radius="${caster_wheel_radius}"/>
+            </geometry>
+            <material name="white"/>
+        </visual>
+        <collision>
+            <geometry>
+                <sphere radius="${caster_wheel_radius}"/>
+            </geometry>
+        </collision>
+        <inertial>
+            <origin xyz="0 0 0" rpy="0 0 0"/>
+            <mass value="${caster_wheel_mass}" />
+            <inertia ixx="${(2/5) * caster_wheel_mass * (caster_wheel_radius*caster_wheel_radius)}" ixy="0.0" ixz="0.0"
+                     iyy="${(2/5) * caster_wheel_mass * (caster_wheel_radius*caster_wheel_radius)}" iyz="0.0"
+                     izz="${(2/5) * caster_wheel_mass * (caster_wheel_radius*caster_wheel_radius)}" />
+        </inertial>
+    </link>
+    <gazebo reference="caster_wheel">
+        <material>Gazebo/White</material>
+        <mu1 value="0.001"/>
+        <mu2 value="0.001"/>
+    </gazebo>
 </robot>

File: ex05/robot_description/urdf/gazebo.urdf.xacro (robot description, xacro)
@@ -2,4 +2,19 @@
 <robot xmlns:xacro="http://www.ros.org/wiki/xacro">
     <gazebo>
+        <!--plugin
+            filename="gz-sim-pose-publisher-system"
+            name="gz::sim::systems::PosePublisher">
+            <publish_link_pose>true</publish_link_pose>
+            <use_pose_vector_msg>true</use_pose_vector_msg>
+            <static_publisher>true</static_publisher>
+            <static_update_frequency>1</static_update_frequency>
+        </plugin-->
+        <!--plugin
+            filename="gz-sim-odometry-publisher-system"
+            name="gz::sim::systems::OdometryPublisher">
+            <odom_frame>robot/odom</odom_frame>
+            <robot_base_frame>robot/base_link</robot_base_frame>
+            <odom_publish_frequency>50</odom_publish_frequency>
+        </plugin-->
         <plugin
             filename="gz-sim-joint-state-publisher-system"
@@ -16,4 +31,11 @@
             <odom_publish_frequency>10</odom_publish_frequency>
         </plugin>
+        <plugin filename="gz-sim-sensors-system"
+                    name="gz::sim::systems::Sensors">
+                <render_engine>ogre2</render_engine>
+        </plugin>
+        <plugin filename="gz-sim-imu-system"
+        name="gz::sim::systems::Imu">
+        </plugin>
     </gazebo>
 </robot>

File: ex05/robot_description/urdf/robot.urdf.xacro (robot description, xacro)
@@ -1,7 +1,8 @@
 <?xml version="1.0" ?>
 <robot name='robot' xmlns:xacro="http://ros.org/wiki/xacro">
-    <xacro:include filename="$(find robot_description)/urdf/gazebo.urdf.xacro" />
-    <!--xacro:include filename="$(find robot_description)/urdf/lidar.urdf.xacro" /-->
-    <!--xacro:include filename="$(find robot_description)/urdf/depth.urdf.xacro" /-->
+    <xacro:include filename="gazebo.urdf.xacro" />
+    <xacro:include filename="lidar.urdf.xacro"/>
+    <xacro:include filename="depth.urdf.xacro" />
+    <xacro:include filename="imu.urdf.xacro" />
     <xacro:property name="chassis_length" value="0.335"/>
     <xacro:property name="chassis_width" value="0.265"/>
@@ -58,5 +59,5 @@
         <origin xyz="${chassis_length/2} 0 ${chassis_height/2}"/>
         <geometry>
-            <cylinder radius="0.1" length="${chassis_height}"/>
+            <box size="${chassis_length} ${chassis_width} ${chassis_height}"/>
         </geometry>
         <material name="orange"/>
@@ -160,21 +161,3 @@
         <mu2 value="0.001"/>
     </gazebo>
-    <link name="sub_spoiler">
-        <visual>
-            <geometry>
-            <cylinder radius="0.05" length="0.2"/>
-        </geometry>
-            <material name="blue"/>
-        </visual>
-        <collision>
-            <geometry>
-                <cylinder radius="0.05" length="0.2"/>
-            </geometry>
-        </collision>
-    </link>
-    <joint name="sub_spoiler_joint" type="fixed">
-        <parent link="base_link"/>
-        <child link="sub_spoiler"/>
-        <origin xyz="0 0 0.10" rpy="0 0 0"/>
-    </joint>
 </robot>
